Commit message: In process of feeding foot contact into the GRF Controller, but have an odd segfault error

File: models/urdf/quadf.urdf (robot description, URDF)
Before this commit: robot quadf, 13 links, 12 joints
Links:
- removed link front right hip 
- added link front right hip, mass 0.594830758051326; collision mesh filename=../meshes/front right hip.obj; visual mesh filename=../meshes/front right hip.obj
Joints:
- joint front right hip joint: child front right hip  -> front right hip
- joint right front UL joint: parent front right hip  -> front right hip

Commit message: The grf controller works better now. If foot contact estimator is used correctly, the quadruped fumbles around and fails to stand

File: models/urdf/quadf.urdf (robot description, URDF)
Before this commit: robot quadf, 13 links, 12 joints
Links:
- added link left back foot, mass 0.0001
- added link left front foot, mass 0.0001
- added link right back foot, mass 0.0001
- added link right front foot, mass 0.0001
Joints:
- added joint left back foot joint: type fixed, parent left back LL, child left back foot, origin xyz=0 0 0.220 rpy=0 0 0, axis 0 0 0
- added joint left front foot joint: type fixed, parent left front LL, child left front foot, origin xyz=0 0 0.220 rpy=0 0 0, axis 0 0 0
- added joint right back foot joint: type fixed, parent right back LL, child right back foot, origin xyz=0 0 0.220 rpy=0 0 0, axis 0 0 0
- added joint right front foot joint: type fixed, parent right front LL, child right front foot, origin xyz=0 0 0.220 rpy=0 0 0, axis 0 0 0
- joint Back left hip joint: origin xyz=-0.125000000000011 -0.310800000000001 -0.0266306081677699 rpy=3.14159265358979 0 -3.14159265358979 -> xyz=-0.15000000000011 -0.310800000000001 -0.0266306081677699 rpy=3.14159265358979 0 -3.14159265358979
- joint Back right hip joint: origin xyz=0.12499999999998 -0.3103 -0.0266306081677744 rpy=0 0 0 -> xyz=0.1499999999998 -0.3103 -0.0266306081677744 rpy=0 0 0
- joint front left hip joint: origin xyz=-0.125000000000013 0.282500000000001 -0.0266306081677672 rpy=0 0 -3.14159265358979 -> xyz=-0.15000000000013 0.282500000000001 -0.0266306081677672 rpy=0 0 -3.14159265358979
- joint front right hip joint: origin xyz=0.124999999999999 0.283000000000001 -0.0266306081677545 rpy=-3.14159265358979 0 0 -> xyz=0.14999999999999 0.283000000000001 -0.0266306081677545 rpy=-3.14159265358979 0 0
- joint left back UL joint: limit lower=-6 upper=6 effort=9 velocity=5 -> (none)
- joint left front UL joint: limit lower=-6 upper=6 effort=9 velocity=5 -> (none)
- joint right back UL joint: limit lower=-6 upper=6 effort=9 velocity=5 -> (none)
- joint right front UL joint: limit lower=-6 upper=6 effort=9 velocity=5 -> (none)
